File: USB2CANv2/USB2CANv2.kicad_sch (KiCad schematic)
At the start: 16 parts, among them SW1 SW_BOOT0, U1 STM32F405RGTx

Commit message: Added most of needed components, from previous scheme.
Parts:
- added C13, C14: 2.2uF, symbol Device:C
- added C5, C6, C7, C8: 22pF, Capacitor_SMD:C_0402_1005Metric_Pad0.74x0.62mm_HandSolder, symbol Device:C_Small
- added H1, H2, H3, H4: MountingHole, symbol Mechanical:MountingHole
- added IC1: MIC5528-3.3YMT-TR, SON40P120X120X60-7N-D, symbol MIC5528-3.3YMT-TR:MIC5528-3.3YMT-TR
- added J1: USB_C_Receptacle_USB2.0, symbol Connector:USB_C_Receptacle_USB2.0
- added J1: STLINK, Connector_PinHeader_2.54mm:PinHeader_1x04_P2.54mm_Vertical, symbol Connector:Conn_01x04_Male
- added R2, R4: 5k1, symbol Device:R
- added R3: 1k5, symbol Device:R
- added R5, R6: 22, symbol Device:R
- added R7: 100, symbol Device:R
- added R8: 1k, symbol Device:R
- added U2: USBLC6-2P6, Package_TO_SOT_SMD:SOT-666, symbol Power_Protection:USBLC6-2P6
- added U3: MCP2561-E-SN, Package_SO:SOIC-8_3.9x4.9mm_P1.27mm, symbol Interface_CAN_LIN:MCP2561-E-SN
- added U4: TLP175A, Package_SO:MFSOP6-4_4.4x3.6mm_P1.27mm, symbol Relay_SolidState:TLP175A
- added Y1: 16MHz, Crystal:Crystal_SMD_5032-2Pin_5.0x3.2mm, symbol Device:Crystal_Small
- added Y2: 32KHz, Crystal:Crystal_SMD_3215-2Pin_3.2x1.5mm, symbol Device:Crystal_Small
Connections:
- net +3.3V: now also C14.1, IC1.1 (VOUT_1), IC1.2 (VOUT_2), R3.2
- net GND: now also C13.2, C14.2, C5.2, C6.2, C7.2, C8.2, IC1.3 (GND), IC1.7 (EP), J1.4 (Pin_4), J1.A1 (GND), J1.A12 (GND), J1.B1 (GND), J1.B12 (GND), J1.S1 (SHIELD), R2.1, R4.1, U3.2 (VSS), U3.8 (STBY), U4.3
- new net: J1.A6 (D+), J1.B6 (D+), R3.1, R5.2
- new net: J1.A5 (CC1), R2.2
- new net: J1.A7 (D-), J1.B7 (D-), R6.2
- new net: J1.B5 (CC2), R4.2
- new net: R8.2, U4.1
- new net: R7.2, U4.6
- new net +5V: C13.1, IC1.4 (EN), IC1.6 (VIN), J1.1 (Pin_1)
- new net CAN_H: R7.1, U3.7 (CANH)
- new net CAN_L: U3.6 (CANL), U4.4
- new net CAN_RX: U3.4 (RXD)
- new net CAN_TX: U3.1 (TXD)
- new net L_OSC_IN: C7.1, Y2.1
- new net L_OSC_OUT: C8.1, Y2.2
- new net OSC_IN: C5.1, Y1.1
- new net OSC_OUT: C6.1, Y1.2
- new net STM_D+: U2.3 (I/O2)
- new net STM_D-: U2.1 (I/O1)
- new net SWCLK: J1.2 (Pin_2)
- new net SWDIO: J1.3 (Pin_3)
- new net TERMINATOR_SIGNAL: R8.1
- new net USB_D+: R5.1, U2.4 (I/O2)
- new net USB_D-: R6.1, U2.6 (I/O1)
- new net USB_VBUS: J1.A4 (VBUS), J1.A9 (VBUS), J1.B4 (VBUS), J1.B9 (VBUS)
- no-connect marks 0 -> 3
Other:
- moved on the sheet: C1, C10, C11, C12, C2, C3, C4, C5, C6, C7, C8, C9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

Commit message: Done scheme
Parts:
- removed J1: STLINK, Connector_PinHeader_2.54mm:PinHeader_1x04_P2.54mm_Vertical, symbol Connector:Conn_01x04_Male
- added D1, D2, D3 (x2): BUILTIN_LED, LED_SMD:LED_0805_2012Metric, symbol Device:LED
- added J3: Conn_01x04_Pin, symbol Connector:Conn_01x04_Pin
- added R10: 100, symbol Device:R
- added R2, R3, R4 (x2): 510, Resistor_SMD:R_0402_1005Metric_Pad0.72x0.64mm_HandSolder, symbol Device:R_Small
- added R9: 1k, symbol Device:R
- added U5: MCP2561-E-SN, Package_SO:SOIC-8_3.9x4.9mm_P1.27mm, symbol Interface_CAN_LIN:MCP2561-E-SN
- added U6: TLP175A, Package_SO:MFSOP6-4_4.4x3.6mm_P1.27mm, symbol Relay_SolidState:TLP175A
Connections:
- net CAN_RX is gone; now on net CAN1_RX: U3.4 (RXD)
- net CAN_TX is gone; now on net CAN1_TX: U3.1 (TXD)
- net L_OSC_IN is gone; now on net HSE_IN: C7.1, Y2.1
- net L_OSC_OUT is gone; now on net HSE_OUT: C8.1, Y2.2
- net OSC_IN is gone; now on net LSE_IN: C5.1, Y1.1
- net OSC_OUT is gone; now on net LSE_OUT: C6.1, Y1.2
- net TERMINATOR_SIGNAL is gone; now on net TERMINATOR_CAN2: R8.1
- net USB_VBUS is gone; now on net +5V: J1.A4 (VBUS), J1.A9 (VBUS), J1.B4 (VBUS), J1.B9 (VBUS)
- net +3.3V: now also D1.2 (A), D2.2 (A), D3.2 (A), D3.2 (A)
- net +5V: now also U2.5 (VBUS), U3.3 (VDD), J3.4 (Pin_4), U5.3 (VDD)
- net GND: now also U2.2 (GND), J3.1 (Pin_1), U5.2 (VSS), U5.8 (STBY), U6.3
- net STM_D+: now also U1.45 (PA12)
- net STM_D-: now also U1.44 (PA11)
- net SWCLK: now also U1.49 (PA14), J3.2 (Pin_2)
- net SWDIO: now also U1.46 (PA13), J3.3 (Pin_3)
- net LED_CAN2: now reaches U1.10 (PC2)
- net LED_CAN2: now also R2.2
- net LED_UART: now reaches U1.11 (PC3)
- net LED_UART: now also R4.2
- net STATUS_LED: now reaches U1.24 (PC4)
- net STATUS_LED: now also R4.2
- net TERMINATOR_CAN2: now reaches U1.29 (PB10)
- net LSE_IN: now reaches U1.3 (PC14)
- net TERMINATOR_CAN1: now reaches U1.30 (PB11)
- net TERMINATOR_CAN1: now also R9.1
- net LSE_OUT: now reaches U1.4 (PC15)
- net HSE_IN: now reaches U1.5 (PH0)
- net SWO: now reaches U1.55 (PB3)
- net CAN2_RX: now reaches U1.57 (PB5)
- net CAN2_RX: now also U5.4 (RXD)
- net CAN2_TX: now reaches U1.58 (PB6)
- net CAN2_TX: now also U5.1 (TXD)
- net HSE_OUT: now reaches U1.6 (PH1)
- net CAN1_RX: now reaches U1.61 (PB8)
- net CAN1_TX: now reaches U1.62 (PB9)
- net LED_CAN1: now reaches U1.9 (PC1)
- net LED_CAN1: now also R3.2
- net CAN_H renamed CAN1_H
- net CAN1_H: now also R10.1; no longer R7.1
- net CAN_L renamed CAN1_L
- net CAN1_L: now also U6.4; no longer U4.4
- new net: D3.1 (K), R4.1 (x2)
- new net: R9.2, U6.1
- new net: R10.2, U6.6
- new net: D1.1 (K), R2.1
- new net: D2.1 (K), R3.1
- new net CAN2_H: R7.1, U5.7 (CANH)
- new net CAN2_L: U4.4, U5.6 (CANL)
- no-connect marks 3 -> 38
Other:
- note added: "CAN 1 Translator"
- note added: "CAN 2 Translator"
- note added: "ESD PROTECTION"
- note added: "HSE OSCILLATOR"
- note added: "LDO 5V to 3.3V"
- note added: "LED'S"
- note added: "LSE OSCILLATOR"
- note added: "MOUNTING HOLES"
- note added: "Microcontroller STM32"
- note added: "SWD DEBUG"
- note added: "Terminator CAN 1"
- note added: "Terminator CAN 2"
- note added: "USB C"
- company: (none) -> Gdańsk PGRacingTeam
- title: (none) -> USB2CAN- CAN TO UART TRANSLATION
- moved on the sheet: C1, C10, C11, C12, C13, C14, C2, C3, C4, C5, C6, C7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

Commit message: Footprints added
Parts:
- C13, C14: footprint (none) -> Capacitor_SMD:C_0402_1005Metric
- H1, H2, H3, H4: footprint (none) -> MountingHole:MountingHole_2.1mm
- IC1: footprint SON40P120X120X60-7N-D -> MIC5528-3.3YMT-TR:SON40P120X120X60-7N-D
- J1: footprint (none) -> Connector_USB:USB_C_Receptacle_GCT_USB4085
- J3: footprint (none) -> Connector_PinHeader_2.54mm:PinHeader_1x01_P2.54mm_Vertical
- R10, R2, R3, R4, R5, R6, R7, R8, R9: footprint (none) -> Resistor_SMD:R_0603_1608Metric
Changed lines of the file:
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@@
       (effects (font (size 1.27 1.27)) (justify left))
     )
-    (property "Footprint" "" (at 263.525 110.49 0)
+    (property "Footprint" "MountingHole:MountingHole_2.1mm" (at 263.525 110.49 0)
       (effects (font (size 1.27 1.27)) hide)
     )
@@
       (effects (font (size 1.27 1.27)))
     )
-    (property "Footprint" "" (at 236.982 62.23 90)
+    (property "Footprint" "Resistor_SMD:R_0603_1608Metric" (at 236.982 62.23 90)
       (effects (font (size 1.27 1.27)) hide)
     )
@@
       (effects (font (size 1.27 1.27)))
     )
-    (property "Footprint" "" (at 231.14 60.198 90)
+    (property "Footprint" "Resistor_SMD:R_0603_1608Metric" (at 231.14 60.198 90)
       (effects (font (size 1.27 1.27)) hide)
     )
@@
       (effects (font (size 1.27 1.27)))
     )
-    (property "Footprint" "" (at 241.3 36.068 90)
+    (property "Footprint" "Resistor_SMD:R_0603_1608Metric" (at 241.3 36.068 90)
       (effects (font (size 1.27 1.27)) hide)
     )
@@
       (effects (font (size 1.27 1.27)) (justify right))
     )
-    (property "Footprint" "" (at 269.24 46.99 0)
+    (property "Footprint" "Connector_USB:USB_C_Receptacle_GCT_USB4085" (at 269.24 46.99 0)
       (effects (font (size 1.27 1.27)) hide)
     )
@@
       (effects (font (size 1.27 1.27)))
     )
-    (property "Footprint" "" (at 231.14 52.578 90)
+    (property "Footprint" "Resistor_SMD:R_0603_1608Metric" (at 231.14 52.578 90)
       (effects (font (size 1.27 1.27)) hide)
     )
@@
       (effects (font (size 1.27 1.27)) (justify right))
     )
-    (property "Footprint" "" (at 161.29 179.07 0)
+    (property "Footprint" "Connector_PinHeader_2.54mm:PinHeader_1x01_P2.54mm_Vertical" (at 161.29 179.07 0)
       (effects (font (size 1.27 1.27)) hide)
     )
@@
       (effects (font (size 1.27 1.27)) (justify left))
     )
-    (property "Footprint" "" (at 240.665 97.79 0)
+    (property "Footprint" "MountingHole:MountingHole_2.1mm" (at 240.665 97.79 0)
       (effects (font (size 1.27 1.27)) hide)
     )
@@
       (effects (font (size 1.27 1.27)) (justify left))
     )
-    (property "Footprint" "" (at 239.522 135.89 90)
+    (property "Footprint" "Resistor_SMD:R_0603_1608Metric" (at 239.522 135.89 90)
       (effects (font (size 1.27 1.27)) hide)
     )
@@
       (effects (font (size 1.27 1.27)) (justify left))
     )
-    (property "Footprint" "" (at 259.842 135.89 90)
+    (property "Footprint" "Resistor_SMD:R_0603_1608Metric" (at 259.842 135.89 90)
       (effects (font (size 1.27 1.27)) hide)
     )
@@
       (effects (font (size 1.27 1.27)) (justify left))
     )
-    (property "Footprint" "" (at 186.182 135.89 90)
+    (property "Footprint" "Resistor_SMD:R_0603_1608Metric" (at 186.182 135.89 90)
       (effects (font (size 1.27 1.27)) hide)
     )
@@
       (effects (font (size 1.27 1.27)))
     )
-    (property "Footprint" "SON40P120X120X60-7N-D" (at 39.37 265.1 0)
+    (property "Footprint" "MIC5528-3.3YMT-TR:SON40P120X120X60-7N-D" (at 39.37 265.1 0)
       (effects (font (size 1.27 1.27)) (justify left top) hide)
     )
@@
       (effects (font (size 1.27 1.27)))
     )
-    (property "Footprint" "" (at 241.3 43.688 90)
+    (property "Footprint" "Resistor_SMD:R_0603_1608Metric" (at 241.3 43.688 90)
       (effects (font (size 1.27 1.27)) hide)
     )
@@
       (effects (font (size 1.27 1.27)) (justify left))
     )
-    (property "Footprint" "" (at 240.665 110.49 0)
+    (property "Footprint" "MountingHole:MountingHole_2.1mm" (at 240.665 110.49 0)
       (effects (font (size 1.27 1.27)) hide)
     )
@@
       (effects (font (size 1.27 1.27)) (justify left))
     )
-    (property "Footprint" "" (at 206.502 135.89 90)
+    (property "Footprint" "Resistor_SMD:R_0603_1608Metric" (at 206.502 135.89 90)
       (effects (font (size 1.27 1.27)) hide)
     )
@@
       (effects (font (size 1.27 1.27)) (justify left))
     )
-    (property "Footprint" "" (at 77.1652 177.8 0)
+    (property "Footprint" "Capacitor_SMD:C_0402_1005Metric" (at 77.1652 177.8 0)
       (effects (font (size 1.27 1.27)) hide)
     )
@@
       (effects (font (size 1.27 1.27)) (justify left))
     )
-    (property "Footprint" "" (at 25.0952 177.8 0)
+    (property "Footprint" "Capacitor_SMD:C_0402_1005Metric" (at 25.0952 177.8 0)
       (effects (font (size 1.27 1.27)) hide)
     )
@@
       (effects (font (size 1.27 1.27)) (justify left))
     )
-    (property "Footprint" "" (at 263.525 97.79 0)
-      (effects (font (size 1.27 1.27)) hide)
-    )
+    (property "Footprint" "MountingHole:MountingHole_2.1mm" (at 263.525 97.79 0)
+      (effects (font (size 1.27 1.27)) hide)
+    )

Commit message: Creating PCB
Parts:
- removed J3: Conn_01x04_Pin, Connector_PinHeader_2.54mm:PinHeader_1x01_P2.54mm_Vertical, symbol Connector:Conn_01x04_Pin
- added J2: Conn_01x06_Pin, IDC:IDC_SMD_3PIN, symbol Connector:Conn_01x06_Pin
- added J3: Conn_01x02_Pin, Connector_PinHeader_2.00mm:PinHeader_1x02_P2.00mm_Vertical, symbol Connector:Conn_01x02_Pin
- added J4, J5: Conn_01x02_Pin, Connector_PinHeader_2.54mm:PinHeader_1x02_P2.54mm_Vertical, symbol Connector:Conn_01x02_Pin
- added R15, R16, R17, R18: 0, Resistor_SMD:R_0402_1005Metric_Pad0.72x0.64mm_HandSolder, symbol Device:R
- added TP1, TP2, TP3, TP4: TestPoint, TestPoint:TestPoint_Pad_1.5x1.5mm, symbol Connector:TestPoint
Connections:
- net +5V: now also J3.1 (Pin_1)
- net CAN1_H: now also J5.1 (Pin_1)
- net CAN1_L: now also J5.2 (Pin_2)
- net CAN1_RX: now also R16.1
- net CAN1_TX: now also R15.1
- net CAN2_H: now also J4.1 (Pin_1)
- net CAN2_L: now also J4.2 (Pin_2)
- net CAN2_RX: now also R18.1
- net CAN2_TX: now also R17.1
- net GND: now also J2.1 (Pin_1)
- net SWCLK: now also J2.2 (Pin_2)
- net SWDIO: now also J2.3 (Pin_3)
- new net: R15.2, TP1.1
- new net: R17.2, TP3.1
- new net: R16.2, TP2.1
- new net: R18.2, TP4.1
- new net DEBUG_5V: J2.6 (Pin_6), J3.2 (Pin_2)
- no-connect marks 38 -> 40
Other:
- note added: "CAN Outputs"
- note added: "Power From DEBUG"
- note added: "SWD DEBUG IDC CONN"
- note removed: "SWD DEBUG"
- moved on the sheet: C5, C6, C7, C8, D1, D2, D3, R2, R3, R4, R7, R8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
